File: pcb/FastNerfController/_autosave-FastNerfController.kicad_pcb (KiCad board)
At the start: 2 copper layers, 66 x 50 mm, 52 parts, among them J1 Conn_01x03, J10 Conn_01x02, J11 Conn_01x01, J12 Conn_01x01, J13 Conn_01x04, J14 Conn_01x04, J15 Conn_01x05, J16 Conn_01x02, J17 Conn_01x02, J18 Conn_01x02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

Commit message: push
Parts:
- added U2: Teensy4.0, teensy.pretty-master:Teensy40, F.Cu at (264.2, 86.4)
Connections:
- J10 pad 2: Net-(J10-Pad2) -> Net-(J10-Pin_2)
- J7 pad 2: Net-(J7-Pad2) -> Net-(J7-Pin_2)
- J8 pad 2: Net-(J8-Pad2) -> Net-(J8-Pin_2)
- J9 pad 2: Net-(J9-Pad2) -> Net-(J9-Pin_2)
- R1 pad 1: Net-(Q1-Pad4) -> Net-(Q1-G)
- R13 pad 1: Net-(Q1-Pad4) -> Net-(Q1-G)
- R14 pad 1: Net-(Q2-Pad4) -> Net-(Q2-G)
- R15 pad 1: Net-(Q3-Pad4) -> Net-(Q3-G)
- R16 pad 1: Net-(Q4-Pad4) -> Net-(Q4-G)
- R2 pad 1: Net-(Q2-Pad4) -> Net-(Q2-G)
- R3 pad 1: Net-(Q3-Pad4) -> Net-(Q3-G)
- R4 pad 1: Net-(Q4-Pad4) -> Net-(Q4-G)
Routing:
- added copper zone on F.Cu, net Net-(J10-Pin_2)
- added copper zone on F.Cu, net Net-(J7-Pin_2)
- added copper zone on F.Cu, net Net-(J8-Pin_2)
- added copper zone on F.Cu, net Net-(J9-Pin_2)
- removed copper zone on F.Cu, net Net-(J10-Pad2)
- removed copper zone on F.Cu, net Net-(J7-Pad2)
- removed copper zone on F.Cu, net Net-(J8-Pad2)
- removed copper zone on F.Cu, net Net-(J9-Pad2)
