File: pcb/FastNerfController/_autosave-FastNerfController.kicad_sch (KiCad schematic)
At the start: 24 parts, among them J1 Conn_01x03, J11 Conn_01x01, J12 Conn_01x01, J13 Conn_01x04, J14 Conn_01x04, J15 Conn_01x05, J2 Conn_01x03, J3 Conn_01x03, J4 Conn_01x03, J5 Conn_01x01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

Commit message: push
Parts:
- U2: footprint (none) -> teensy.pretty-master:Teensy40
Changed lines of the file:
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@@
       (effects (font (size 1.27 1.27)))
     )
-    (property "Footprint" "" (at 3.81 163.83 0)
+    (property "Footprint" "teensy.pretty-master:Teensy40" (at 3.81 163.83 0)
       (effects (font (size 1.27 1.27)) hide)
     )
