File: pcb/FastNerfController/FastNerfController.kicad_pcb (KiCad board)
At the start: 2 copper layers, 66 x 50 mm, 52 parts, among them J1 Conn_01x03, J10 Conn_01x02, J11 Conn_01x01, J12 Conn_01x01, J13 Conn_01x04, J14 Conn_01x04, J15 Conn_01x05, J16 Conn_01x02, J17 Conn_01x02, J18 Conn_01x02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

Commit message: big push
Parts:
- removed C7, C8: 10uF, Capacitor_SMD:C_0805_2012Metric
- removed J10, J9: Conn_01x02, Connector_PinHeader_2.54mm:PinHeader_1x02_P2.54mm_Vertical
- removed Q3, Q4: DMG7430LFG-7, SamacSys_Parts:POWERDI-3333-8
- removed R15, R16: 2.2k, Resistor_SMD:R_0603_1608Metric
- removed R3, R4: 100, Resistor_SMD:R_0603_1608Metric
- removed U1: MUBv1, MUB:MUB_v1
- added U2: Teensy4.0, teensy.pretty-master:Teensy40_SMT, F.Cu at (191.7, 78.0)
- moved R11 27.8 mm to (202.7, 74.7), turned to 180 degrees
- moved R12 27.5 mm to (202.7, 76.3), turned to 180 degrees
- moved C1 3.75 mm to (182.8, 99.8), turned to 180 degrees
- moved C2 2.57 mm to (192.4, 99.8), turned to 0 degrees
Connections:
- J7 pad 2: Net-(J7-Pad2) -> Net-(J7-Pin_2)
- J8 pad 2: Net-(J8-Pad2) -> Net-(J8-Pin_2)
- R1 pad 1: Net-(Q1-Pad4) -> Net-(Q1-G)
- R13 pad 1: Net-(Q1-Pad4) -> Net-(Q1-G)
- R14 pad 1: Net-(Q2-Pad4) -> Net-(Q2-G)
- R2 pad 1: Net-(Q2-Pad4) -> Net-(Q2-G)
Routing:
- net /BLDC 3: track 79.5 -> 24.1 mm, vias 2 -> 0
- net /BLDC 4: track 70.8 -> 15.4 mm, vias 2 -> 0
- net (no net): track 0.00 -> 41.0 mm, vias 0 -> 2
- net /TX: track 45.6 -> 10.6 mm, vias 3 -> 0
- net /RX: track 43.5 -> 9.57 mm, vias 3 -> 0
- net /BTN: track 36.9 -> 3.35 mm
- net /DIR: track 37.3 -> 5.97 mm
- net /Gate4: track 29.9 -> 0.00 mm, vias 2 -> 0
- net /PULSE: track 38.5 -> 9.18 mm
- net /Gate3: track 28.0 -> 0.00 mm, vias 2 -> 0
- net /Button4: track 32.3 -> 5.12 mm
- net /Button3: track 33.2 -> 7.64 mm
- net /BLDC 2: track 58.3 -> 35.4 mm
- net /Button2: track 26.8 -> 4.41 mm
- net /Button1: track 28.3 -> 7.62 mm
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- added copper zone on F.Cu, net Net-(J7-Pin_2)
- added copper zone on F.Cu, net Net-(J8-Pin_2)
- removed copper zone on F.Cu, net Net-(J10-Pad2)
- removed copper zone on F.Cu, net Net-(J7-Pad2)
- removed copper zone on F.Cu, net Net-(J8-Pad2)
- removed copper zone on F.Cu, net Net-(J9-Pad2)
