File: pcb/FastNerfController/FastNerfController.kicad_sch (KiCad schematic)
At the start: 24 parts, among them J1 Conn_01x03, J11 Conn_01x01, J12 Conn_01x01, J13 Conn_01x04, J14 Conn_01x04, J15 Conn_01x05, J2 Conn_01x03, J3 Conn_01x03, J4 Conn_01x03, J5 Conn_01x01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

Commit message: big push
Parts:
- removed U1: MUBv1, MUB:MUB_v1, symbol MUB:MUBv1
- U2: footprint (none) -> teensy.pretty-master:Teensy40_SMT
Connections:
- net +5V: now also U2.33 (VIN)
- net BLDC 1: now also U2.4 (2_OUT2)
- net BLDC 2: now also U2.5 (3_LRCLK2)
- net BLDC 3: now also U2.6 (4_BCLK2)
- net BLDC 4: now also U2.7 (5_IN2)
- net BTN: now also U2.22 (15_A1_RX3_SPDIF_IN)
- net Battery_V: now also U2.21 (14_A0_TX3_SPDIF_OUT)
- net Button1: now also U2.2 (0_RX1_CRX2_CS1)
- net Button2: now also U2.3 (1_TX1_CTX2_MISO1)
- net Button3: now also U2.13 (11_MOSI_CTX1)
- net Button4: now also U2.14 (12_MISO_MQSL)
- net DIR: now also U2.23 (16_A2_RX4_SCL1)
- net GND: now also U2.1 (GND), U2.32 (GND)
- net Gate1: now also U2.11 (9_OUT1C)
- net Gate2: now also U2.12 (10_CS_MQSR)
- net PULSE: now also U2.24 (17_A3_TX4_SDA1)
- net SCL: now also U2.26 (19_A5_SCL0)
- net SDA: now also U2.25 (18_A4_SDA0)
- net at U2.10 (8_TX2_IN1): now also R12.2
- net at U2.9 (7_RX2_OUT1A): now also R11.2
Other:
- removed sheet DC Driver 3
- removed sheet DC Driver 4
- moved on the sheet: R11, R12, U2
